Commit message: added https://github.com/yzrobot/adaptive_clusterin

File: src/jackal_velodyne/urdf/jackal_velodyne.urdf.xacro (robot description, xacro)
@@ -179,5 +179,5 @@
   <xacro:include filename="$(find velodyne_description)/urdf/VLP-16.urdf.xacro"/>
   <VLP-16 parent="base_link" name="velodyne" topic="/velodyne_points" hz="10" samples="360" gpu="true" lasers="16" max_range="100">
-    <origin xyz="0 0 0.4" rpy="0 0 0" />
+    <origin xyz="0 0 1" rpy="0 0 0" />
   </VLP-16>
   <!-- VHDL-32E -->
